File: ROTO.kicad_sch (KiCad schematic)
At the start: 7 parts, among them J1 POWER INPUT, J2 RELAY, J3 SWITCH, U1 LM7805, U2 SX1509

Commit message: Flipped PCB
Parts:
- removed J3: SWITCH, TerminalBlock_Phoenix:TerminalBlock_Phoenix_MKDS-1,5-9_1x09_P5.00mm_Horizontal, symbol Connector:Screw_Terminal_01x09
- added J3: Switch, TerminalBlock_Phoenix:TerminalBlock_Phoenix_MKDS-1,5-10_1x10_P5.00mm_Horizontal, symbol Connector:Screw_Terminal_01x10
Connections:
- net +5V: now also C1.2; no longer C1.1
- net GND: now also J3.2 (Pin_2); no longer U2.25 (GND)
- net at U1.3 (VO): now also C1.1; no longer C1.2
- net at U2.12 (8): now also J3.10 (Pin_10)
- net at U2.13 (9): now also J3.9 (Pin_9)
- net at U2.14 (10): now also J3.8 (Pin_8)
- net at U2.15 (11): now also J3.7 (Pin_7)
- net at U2.16 (12): now also J3.6 (Pin_6)
- net at U2.17 (13): now also J3.5 (Pin_5)
- net at U2.18 (14): now also J3.4 (Pin_4)
- net at U2.19 (15): now also J3.3 (Pin_3)
- no-connect marks 29 -> 36
Other:
- moved on the sheet: C1
Changed lines of the file:
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@@
   (junction (at 30.48 105.41) (diameter 0) (color 0 0 0 0)
-  )
-  (junction (at 209.55 114.3) (diameter 0) (color 0 0 0 0)
   )
   (no_connect (at 203.2 97.79))
@@
   (no_connect (at 160.02 96.52))
   (no_connect (at 129.54 95.25))
+  (no_connect (at 222.25 114.3))
   (no_connect (at 231.14 105.41))
   (no_connect (at 93.98 102.87))
   (no_connect (at 93.98 87.63))
+  (no_connect (at 210.82 80.01))
   (no_connect (at 231.14 100.33))
   (no_connect (at 93.98 110.49))
@@
   (no_connect (at 203.2 93.98))
   (no_connect (at 93.98 95.25))
+  (no_connect (at 217.17 114.3))
   (no_connect (at 93.98 105.41))
   (no_connect (at 160.02 101.6))
@@
   (no_connect (at 195.58 96.52))
   (no_connect (at 129.54 92.71))
+  (no_connect (at 227.33 114.3))
   (no_connect (at 195.58 104.14))
   (no_connect (at 203.2 90.17))
+  (no_connect (at 217.17 80.01))
   (no_connect (at 160.02 99.06))
+  (no_connect (at 271.78 77.47))
+  (no_connect (at 207.01 114.3))
   (no_connect (at 93.98 107.95))
   (no_connect (at 231.14 93.98))
@@
     (stroke (width 0) (type default))
   )
+  (wire (pts (xy 269.24 81.28) (xy 270.51 81.28))
+    (stroke (width 0) (type default))
+  )
   (wire (pts (xy 256.54 82.55) (xy 256.54 77.47))
     (stroke (width 0) (type default))
@@
     (stroke (width 0) (type default))
   )
-  (wire (pts (xy 209.55 114.3) (xy 212.09 114.3))
-    (stroke (width 0) (type default))
-  )
   (wire (pts (xy 195.58 99.06) (xy 200.66 99.06))
     (stroke (width 0) (type default))
@@
     (stroke (width 0) (type default))
   )
-  (wire (pts (xy 209.55 114.3) (xy 209.55 118.11))
+  (wire (pts (xy 212.09 114.3) (xy 212.09 118.11))
     (stroke (width 0) (type default))
   )
@@
     (stroke (width 0) (type default))
   )
-  (wire (pts (xy 207.01 114.3) (xy 209.55 114.3))
-    (stroke (width 0) (type default))
-  )
   (wire (pts (xy 270.51 113.03) (xy 271.78 113.03))
     (stroke (width 0) (type default))
@@
     (stroke (width 0) (type default))
   )
-  (wire (pts (xy 264.16 82.55) (xy 264.16 77.47))
+  (wire (pts (xy 269.24 81.28) (xy 269.24 77.47))
+    (stroke (width 0) (type default))
+  )
+  (wire (pts (xy 264.16 77.47) (xy 264.16 82.55))
     (stroke (width 0) (type default))
   )
@@
     (stroke (width 0) (type default))
   )
-  (wire (pts (xy 254 82.55) (xy 254 77.47))
-    (stroke (width 0) (type default))
-  )
-  (wire (pts (xy 269.24 77.47) (xy 270.51 78.74))
+  (wire (pts (xy 254 77.47) (xy 254 82.55))
     (stroke (width 0) (type default))
   )
@@
     )
   )
-  (symbol (lib_id "Device:C") (at 36.83 105.41 90) (unit 1)
-    (in_bom yes) (on_board yes) (dnp no) (fields_autoplaced)
-    (property "Reference" "C1" (at 36.83 99.06 90)
-      (effects (font (size 1.27 1.27)))
-    )
-    (property "Value" "C" (at 36.83 101.6 90)
-      (effects (font (size 1.27 1.27)))
-    )
-    (property "Footprint" "Capacitor_THT:C_Radial_D4.0mm_H7.0mm_P1.50mm" (at 40.64 104.4448 0)
+  (symbol (lib_id "Device:C") (at 36.83 105.41 270) (mirror x) (unit 1)
+    (in_bom yes) (on_board yes) (dnp no)
+    (property "Reference" "C1" (at 36.83 113.03 90)
+      (effects (font (size 1.27 1.27)))
+    )
+    (property "Value" "C" (at 36.83 110.49 90)
+      (effects (font (size 1.27 1.27)))
+    )
+    (property "Footprint" "Capacitor_THT:C_Radial_D4.0mm_H7.0mm_P1.50mm" (at 33.02 104.4448 0)
       (effects (font (size 1.27 1.27)) hide)
     )
@@
     )
   )
-  (symbol (lib_id "power:GND") (at 270.51 78.74 90) (unit 1)
-    (in_bom yes) (on_board yes) (dnp no)
-    (property "Reference" "#PWR05" (at 276.86 78.74 0)
-      (effects (font (size 1.27 1.27)) hide)
-    )
-    (property "Value" "GND" (at 273.05 82.55 90)
-      (effects (font (size 1.27 1.27)))
-    )
-    (property "Footprint" "" (at 270.51 78.74 0)
-      (effects (font (size 1.27 1.27)) hide)
-    )
-    (property "Datasheet" "" (at 270.51 78.74 0)
+  (symbol (lib_id "power:GND") (at 270.51 81.28 90) (unit 1)
+    (in_bom yes) (on_board yes) (dnp no)
+    (property "Reference" "#PWR05" (at 276.86 81.28 0)
+      (effects (font (size 1.27 1.27)) hide)
+    )
+    (property "Value" "GND" (at 273.05 85.09 90)
+      (effects (font (size 1.27 1.27)))
+    )
+    (property "Footprint" "" (at 270.51 81.28 0)
+      (effects (font (size 1.27 1.27)) hide)
+    )
+    (property "Datasheet" "" (at 270.51 81.28 0)
       (effects (font (size 1.27 1.27)) hide)
     )
@@
     )
   )
-  (symbol (lib_id "power:GND") (at 209.55 118.11 0) (unit 1)
-    (in_bom yes) (on_board yes) (dnp no) (fields_autoplaced)
-    (property "Reference" "#PWR010" (at 209.55 124.46 0)
-      (effects (font (size 1.27 1.27)) hide)
-    )
-    (property "Value" "GND" (at 209.55 123.19 0)
-      (effects (font (size 1.27 1.27)))
-    )
-    (property "Footprint" "" (at 209.55 118.11 0)
-      (effects (font (size 1.27 1.27)) hide)
-    )
-    (property "Datasheet" "" (at 209.55 118.11 0)
+  (symbol (lib_id "power:GND") (at 212.09 118.11 0) (unit 1)
+    (in_bom yes) (on_board yes) (dnp no) (fields_autoplaced)
+    (property "Reference" "#PWR010" (at 212.09 124.46 0)
+      (effects (font (size 1.27 1.27)) hide)
+    )
+    (property "Value" "GND" (at 212.09 123.19 0)
+      (effects (font (size 1.27 1.27)))
+    )
+    (property "Footprint" "" (at 212.09 118.11 0)
+      (effects (font (size 1.27 1.27)) hide)
+    )
+    (property "Datasheet" "" (at 212.09 118.11 0)
       (effects (font (size 1.27 1.27)) hide)
     )
@@
     )
   )
-  (symbol (lib_id "Connector:Screw_Terminal_01x09") (at 259.08 72.39 90) (unit 1)
-    (in_bom yes) (on_board yes) (dnp no)
-    (property "Reference" "J3" (at 259.08 66.04 90)
-      (effects (font (size 1.27 1.27)) (justify left))
-    )
-    (property "Value" "SWITCH" (at 261.62 68.58 90)
-      (effects (font (size 1.27 1.27)) (justify left))
-    )
-    (property "Footprint" "TerminalBlock_Phoenix:TerminalBlock_Phoenix_MKDS-1,5-9_1x09_P5.00mm_Horizontal" (at 259.08 72.39 0)
-      (effects (font (size 1.27 1.27)) hide)
-    )
-    (property "Datasheet" "~" (at 259.08 72.39 0)
-      (effects (font (size 1.27 1.27)) hide)
-    )
-    (pin "1")
+  (symbol (lib_id "Connector:Screw_Terminal_01x10") (at 261.62 72.39 270) (mirror x) (unit 1)
+    (in_bom yes) (on_board yes) (dnp no)
+    (property "Reference" "J3" (at 260.35 66.04 90)
+      (effects (font (size 1.27 1.27)))
+    )
+    (property "Value" "Switch" (at 260.35 68.58 90)
+      (effects (font (size 1.27 1.27)))
+    )
+    (property "Footprint" "TerminalBlock_Phoenix:TerminalBlock_Phoenix_MKDS-1,5-10_1x10_P5.00mm_Horizontal" (at 261.62 72.39 0)
+      (effects (font (size 1.27 1.27)) hide)
+    )
+    (property "Datasheet" "~" (at 261.62 72.39 0)
+      (effects (font (size 1.27 1.27)) hide)
+    )
+    (pin "1")
+    (pin "10")
     (pin "2")
     (pin "3")
